File: kicad/guillotine-pcb.kicad_sch (KiCad schematic)
At the start: 82 parts, among them J1 24V POWER (JST-XH), J2 DC MOTOR (JST-XH), J3 CAN (JST-XH), J4 USB-C PROGRAM/DFU, J5 I2C SOLDERABLE HEADER, J6 SPI SOLDERABLE HEADER, J7 SWD PROGRAM HEADER, SW1 RESET, SW2 BOOT/DFU, U1 STM32F072C8T6, U2 AP63205WU-7 (5V/2A), U3 AMS1117-3.3, U4 DRV8870DDAR 3.6A H-bridge, U5 INA180A1IDBVR (20V/V), U6 MT9105ET analog Hall 5mV/G, U7 USBLC6-2SC6 USB ESD, U8 SN65HVD230DR 3.3V CAN, U9 SN74AHCT1G125DBVR, Y1 8MHz 20pF

Commit message: Fully corrected schematic
Parts:
- removed C26, C27, C28, C29: 100nF, Capacitor_SMD:C_0402_1005Metric, symbol Device:C_Small
- removed D4, D5: WS2812B-2020 EDGE, LED_SMD:LED_WS2812B-2020_PLCC4_2.0x2.0mm, symbol LED:WS2812B-2020
- added C35: 47uF 35V, Capacitor_SMD:CP_Elec_6.3x7.7, symbol Device:C_Polarized_Small
- added C36, C37, C38: 100nF, Capacitor_SMD:C_0402_1005Metric, symbol Device:C_Small
- added D11, D12: WS2812B-2020 EDGE, LED_SMD:LED_WS2812B-2020_PLCC4_2.0x2.0mm, symbol LED:WS2812B-2020
- C18: value 10nF VREF filter -> 10nF
- U6: value MT9105ET analog Hall 5mV/G -> MT9105ET; footprint Package_TO_SOT_SMD:SOT-23 -> Package_TO_SOT_SMD:SOT-23W
Connections:
- net NEOPIXEL_D3_TO_D4 is gone; now on an unnamed net: D6.3 (DIN)
- net 24V_RAW: now also C35.1; no longer C19.1, C20.1, U4.5 (VM)
- net CAN_H: now also R13.2; no longer R13.1
- net CAN_L: now also JP1.1 (A); no longer JP1.2 (B)
- net I2C1_SCL_PB6: now also R15.1; no longer R15.2
- net I2C1_SDA_PB7: now also R16.1; no longer R16.2
- net MOTOR_CURRENT_ADC_1V_PER_A: now also C21.2; no longer C21.1
- net MOTOR_VREF_1V1: now also R3.1, R4.2; no longer R3.2, R4.1
- net NRST: now also SW1.2; no longer SW1.1
- net USB_DM_ESD: no longer U7.4 (I/O2)
- net USB_DM_PA11: no longer R11.2
- net USB_DP_ESD: no longer U7.6 (I/O1)
- net USB_DP_PA12: no longer R10.2
- net at D10.1 (DOUT): now also D11.3 (DIN)
- net 3V3_ANALOG renamed +3V3A
- net 3V3_SYS renamed +3V3
- net +3V3: now also C14.2, C22.2, C25.2, R15.2, R16.2; no longer C14.1, C22.1, C25.1, R15.1, R16.1, R3.1
- net 5V_SYS renamed +5V
- net +5V: now also C30.2, C31.2, C32.2, C33.2, C34.2, C36.2, C37.2, C38.2, D11.4 (VDD), D12.4 (VDD); no longer C30.1, C31.1, C32.1, C33.1, C34.1
- removed net CAN_TERM_JUMPER: JP1.1 (A), R13.2
- net GND_0V renamed GND
- net GND: now also C14.1, C21.1, C22.1, C25.1, C30.1, C31.1, C32.1, C33.1, C34.1, R4.1, SW1.1, C35.2, C36.1, C37.1, C38.1, D11.2 (VSS), D12.2 (VSS); no longer C14.2, C21.2, C22.2, C25.2, C30.2, C31.2, C32.2, C33.2, C34.2, R4.2, SW1.2
- net N$1: no longer names the net of J4.A5 (CC1), R8.1
- net N$2: no longer names the net of J4.B5 (CC2), R9.1
- net NEOPIXEL_D1_TO_D2: no longer names the net of D3.1 (DOUT)
- net NEOPIXEL_D4_TO_D5: no longer names the net of D6.1 (DOUT), D7.3 (DIN)
- net NEOPIXEL_D5_TO_D6: no longer names the net of D7.1 (DOUT), D8.3 (DIN)
- net NEOPIXEL_D6_TO_D7: no longer names the net of D8.1 (DOUT), D9.3 (DIN)
- net NEOPIXEL_D7_TO_D8: no longer names the net of D10.3 (DIN), D9.1 (DOUT)
- net USB_DM_CONN: no longer names the net of J4.A7 (D-), J4.B7 (D-)
- net USB_DM_CONN: now also U7.1 (I/O1); no longer U7.3 (I/O2)
- net USB_DP_CONN: no longer names the net of J4.A6 (D+), J4.B6 (D+)
- net USB_DP_CONN: now also U7.3 (I/O2); no longer U7.1 (I/O1)
- new net: R10.2, U7.4 (I/O2)
- new net: R11.2, U7.6 (I/O1)
- new net: JP1.2 (B), R13.1
- new net: D11.1 (DOUT), D12.3 (DIN)
- new net +24V_RAW: C19.1, C20.1, R3.2, U4.5 (VM)
Other:
- company: (none) -> Massive Dynamic
- title: 24 V Electronic Filament Cutter Controller -> Guillotine Electronic Filament Cutter Controller
- moved on the sheet: C1, C10, C11, C12, C13, C14, C15, C16, C17, C18, C19, C2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
